File: 6530 to 6532 adaptor.kicad_sch (KiCad schematic)
At the start: 29 parts, among them J1 IC5, J2 IC5, J3 IC3, J4 IC6, J5 IC6, Q1 2N7000, U10 74LS00, U2 6532, U4 6532, U6 74LS00, U7 74LS11, U8 27C64, U9 74LS42

Commit message: Update name on schematic
Other:
- title: Allied Leisure 6530 to 6530 adaptor with ROM -> Allied Leisure 6530 to 6532 adaptor with ROM
